Commit message: Updated bash file to run everything
Fixed Gripper pos
Displaying marker
Updated Sync

File: mycobot_description/urdf/robots/mycobot_280.urdf.xacro (robot description, xacro)
@@ -40,5 +40,5 @@
                 parent="$(arg flange_link)"
                 prefix="$(arg prefix)">
-                <origin xyz="0 0 0.034" rpy="1.579 0 0"/>
+                <origin xyz="0 0 0.034" rpy="1.579 0 -0.785"/>
             </xacro:adaptive_gripper>
         </xacro:if>
