Commit message: Updated joint limits, I think the grippe needs updating to

File: mycobot_description/urdf/mech/mycobot_280_arm.urdf.xacro (robot description, xacro)
@@ -146,5 +146,5 @@
     <joint name="${prefix}link1_to_${prefix}link2" type="revolute">
       <axis xyz="0 0 1"/>
-      <limit effort="${joint_effort}" lower="-2.879793" upper="2.879793" velocity="${joint_velocity}"/>
+      <limit effort="${joint_effort}" lower = "-2.9322" upper = "2.9322" velocity="${joint_velocity}"/>
       <parent link="${prefix}link1"/>
       <child link="${prefix}link2"/>
@@ -154,5 +154,5 @@
     <joint name="${prefix}link2_to_${prefix}link3" type="revolute">
       <axis xyz="0 0 1"/>
-      <limit effort="${joint_effort}" lower="-2.879793" upper="2.879793" velocity="${joint_velocity}"/>
+      <limit effort="${joint_effort}" lower = "-2.3562" upper = "2.3562" velocity="${joint_velocity}"/>
       <parent link="${prefix}link2"/>
       <child link="${prefix}link3"/>
@@ -162,5 +162,5 @@
     <joint name="${prefix}link3_to_${prefix}link4" type="revolute">
       <axis xyz="0 0 1"/>
-      <limit effort="${joint_effort}" lower="-2.879793" upper="2.879793" velocity="${joint_velocity}"/>
+      <limit effort="${joint_effort}" lower = "-2.618" upper = "2.618" velocity="${joint_velocity}"/>
       <parent link="${prefix}link3"/>
       <child link="${prefix}link4"/>
@@ -170,5 +170,5 @@
     <joint name="${prefix}link4_to_${prefix}link5" type="revolute">
       <axis xyz="0 0 1"/>
-      <limit effort="${joint_effort}" lower="-2.879793" upper="2.879793" velocity="${joint_velocity}"/>
+      <limit effort="${joint_effort}" lower = "-2.5307" upper = "2.5307" velocity="${joint_velocity}"/>
       <parent link="${prefix}link4"/>
       <child link="${prefix}link5"/>
@@ -178,5 +178,5 @@
     <joint name="${prefix}link5_to_${prefix}link6" type="revolute">
       <axis xyz="0 0 1"/>
-      <limit effort="${joint_effort}" lower="-2.879793" upper="2.879793" velocity="${joint_velocity}"/>
+      <limit effort="${joint_effort}" lower = "-2.8798" upper = "2.8798" velocity="${joint_velocity}"/>
       <parent link="${prefix}link5"/>
       <child link="${prefix}link6"/>

Commit message: Updated limits

File: mycobot_description/urdf/mech/mycobot_280_arm.urdf.xacro (robot description, xacro)
@@ -146,5 +146,5 @@
     <joint name="${prefix}link1_to_${prefix}link2" type="revolute">
       <axis xyz="0 0 1"/>
-      <limit effort="${joint_effort}" lower = "-2.9322" upper = "2.9322" velocity="${joint_velocity}"/>
+      <limit effort="${joint_effort}" lower = "-2.879793" upper = "2.879793" velocity="${joint_velocity}"/>
       <parent link="${prefix}link1"/>
       <child link="${prefix}link2"/>
@@ -154,5 +154,5 @@
     <joint name="${prefix}link2_to_${prefix}link3" type="revolute">
       <axis xyz="0 0 1"/>
-      <limit effort="${joint_effort}" lower = "-2.3562" upper = "2.3562" velocity="${joint_velocity}"/>
+      <limit effort="${joint_effort}" lower = "-2.879793" upper = "2.879793" velocity="${joint_velocity}"/>
       <parent link="${prefix}link2"/>
       <child link="${prefix}link3"/>
@@ -162,5 +162,5 @@
     <joint name="${prefix}link3_to_${prefix}link4" type="revolute">
       <axis xyz="0 0 1"/>
-      <limit effort="${joint_effort}" lower = "-2.618" upper = "2.618" velocity="${joint_velocity}"/>
+      <limit effort="${joint_effort}" lower = "-2.879793" upper = "2.879793" velocity="${joint_velocity}"/>
       <parent link="${prefix}link3"/>
       <child link="${prefix}link4"/>
@@ -170,5 +170,5 @@
     <joint name="${prefix}link4_to_${prefix}link5" type="revolute">
       <axis xyz="0 0 1"/>
-      <limit effort="${joint_effort}" lower = "-2.5307" upper = "2.5307" velocity="${joint_velocity}"/>
+      <limit effort="${joint_effort}" lower = "-2.879793" upper = "2.879793" velocity="${joint_velocity}"/>
       <parent link="${prefix}link4"/>
       <child link="${prefix}link5"/>
@@ -178,5 +178,5 @@
     <joint name="${prefix}link5_to_${prefix}link6" type="revolute">
       <axis xyz="0 0 1"/>
-      <limit effort="${joint_effort}" lower = "-2.8798" upper = "2.8798" velocity="${joint_velocity}"/>
+      <limit effort="${joint_effort}" lower = "-2.879793" upper = "2.879793" velocity="${joint_velocity}"/>
       <parent link="${prefix}link5"/>
       <child link="${prefix}link6"/>
