Commit message: Updated paths and a place holder

File: mycobot_description/urdf/control/mycobot_280_ros2_control.urdf.xacro (robot description, xacro)
@@ -17,6 +17,6 @@
             <joint name="${prefix}link2_to_${prefix}link3">
                 <command_interface name="position">
-                    <param name="min">-2.879793</param>
-                    <param name="max">2.879793</param>
+                    <param name="min">-2.356</param>
+                    <param name="max">2.356</param>
                 </command_interface>
                 <state_interface name="position"/>
@@ -24,6 +24,6 @@
             <joint name="${prefix}link3_to_${prefix}link4">
                 <command_interface name="position">
-                    <param name="min">-2.879793</param>
-                    <param name="max">2.879793</param>
+                    <param name="min">-2.618</param>
+                    <param name="max">2.618</param>
                 </command_interface>
                 <state_interface name="position"/>
@@ -31,6 +31,6 @@
             <joint name="${prefix}link4_to_${prefix}link5">
                 <command_interface name="position">
-                    <param name="min">-2.879793</param>
-                    <param name="max">2.879793</param>
+                    <param name="min">-2.530</param>
+                    <param name="max">2.530</param>
                 </command_interface>
                 <state_interface name="position"/>
@@ -38,6 +38,6 @@
             <joint name="${prefix}link5_to_${prefix}link6">
                 <command_interface name="position">
-                    <param name="min">-2.879793</param>
-                    <param name="max">2.879793</param>
+                    <param name="min">-2.880</param>
+                    <param name="max">2.880</param>
                 </command_interface>
                 <state_interface name="position"/>

File: mycobot_description/urdf/mech/mycobot_280_arm.urdf.xacro (robot description, xacro)
@@ -154,5 +154,5 @@
     <joint name="${prefix}link2_to_${prefix}link3" type="revolute">
       <axis xyz="0 0 1"/>
-      <limit effort="${joint_effort}" lower = "-2.879793" upper = "2.879793" velocity="${joint_velocity}"/>
+      <limit effort="${joint_effort}" lower = "-2.356" upper = "2.356" velocity="${joint_velocity}"/>
       <parent link="${prefix}link2"/>
       <child link="${prefix}link3"/>
@@ -162,5 +162,5 @@
     <joint name="${prefix}link3_to_${prefix}link4" type="revolute">
       <axis xyz="0 0 1"/>
-      <limit effort="${joint_effort}" lower = "-2.879793" upper = "2.879793" velocity="${joint_velocity}"/>
+      <limit effort="${joint_effort}" lower = "-2.618" upper = "2.618" velocity="${joint_velocity}"/>
       <parent link="${prefix}link3"/>
       <child link="${prefix}link4"/>
@@ -170,5 +170,5 @@
     <joint name="${prefix}link4_to_${prefix}link5" type="revolute">
       <axis xyz="0 0 1"/>
-      <limit effort="${joint_effort}" lower = "-2.879793" upper = "2.879793" velocity="${joint_velocity}"/>
+      <limit effort="${joint_effort}" lower = "-2.530" upper = "2.530" velocity="${joint_velocity}"/>
       <parent link="${prefix}link4"/>
       <child link="${prefix}link5"/>
@@ -178,5 +178,5 @@
     <joint name="${prefix}link5_to_${prefix}link6" type="revolute">
       <axis xyz="0 0 1"/>
-      <limit effort="${joint_effort}" lower = "-2.879793" upper = "2.879793" velocity="${joint_velocity}"/>
+      <limit effort="${joint_effort}" lower = "-2.880" upper = "2.880" velocity="${joint_velocity}"/>
       <parent link="${prefix}link5"/>
       <child link="${prefix}link6"/>
